Commit message: Modified urdf and visualizer to show snake correctly

File: reusnake_visualize/urdf/rotary_module.xacro (robot description, xacro)
@@ -3,9 +3,9 @@
   <xacro:property name="mass_2" value=".103" />
   <xacro:property name="cyl_r" value=".026" />
-  <xacro:property name="cyl_h" value=".033" />
+  <xacro:property name="cyl_h" value="-0.033" />
   <xacro:macro name="rotary_module_in" params="name">
     <link name="${name}">
       <visual>
-	<origin xyz="0 0 0.035" rpy="1.57075 0 0" />
+	<origin xyz="0 0 -0.035" rpy="-1.57075 0 0" />
         <geometry>
           <mesh filename="package://reusnake_visualize/meshes/rotary_input.stl"/>
@@ -14,5 +14,5 @@
       </visual>
     <collision>
-      <origin xyz="0 0 ${0.0366/2.0}" rpy="0 0 0" />
+      <origin xyz="0 0 -${0.0366/2.0}" rpy="0 0 0" />
       <geometry>
 	<cylinder radius="${cyl_r}" length="${cyl_h}" />
@@ -20,5 +20,5 @@
     </collision>
     <inertial>
-      <origin xyz="0 0 0.0366" rpy="0 0 0" />
+      <origin xyz="0 0 -0.0366" rpy="0 0 0" />
       <mass value="${mass_2}"/>
       <inertia ixx="${mass_2/12.0*(3*cyl_r**2+cyl_h**2)+mass_2*(cyl_h/2.0)**2}" iyy="${mass_2/12.0*(3*cyl_r**2+cyl_h**2)+mass_2*(cyl_h/2.0)**2}" izz="${mass_2/2.0*cyl_r**2}" ixy="0" ixz="0" iyz="0" />
@@ -30,5 +30,5 @@
       <parent link="${parent}"/>
       <child link="${child}"/>
-      <origin xyz="0 0 0.0366" rpy="0 0 0"/>
+      <origin xyz="0 0 -0.0366" rpy="0 0 0"/>
       <axis xyz="0 1 0"/>
       <dynamics damping=".1" friction="0.2"/>
@@ -49,5 +49,5 @@
     <link name="${name}">
       <visual>
-        <origin xyz="0 0 0" rpy="1.57075 0 0" />
+        <origin xyz="0 0 0" rpy="-1.57075 0 0" />
         <geometry>
           <mesh filename="package://reusnake_visualize/meshes/rotary_output.stl"/>
@@ -57,5 +57,5 @@
       </visual>
     <collision>
-      <origin xyz="0 0 ${0.0366/2.0}" rpy="0 0 0" />
+      <origin xyz="0 0 -${0.0366/2.0}" rpy="0 0 0" />
       <geometry>
 	<cylinder radius="${cyl_r}" length="${cyl_h}" />
@@ -73,5 +73,5 @@
       <parent link="${parent}"/>
       <child link="${child}"/>
-      <origin xyz="0 0 0.0273" rpy="0 0 -1.57075"/>
+      <origin xyz="0 0 -0.0273" rpy="0 0 -1.57075"/>
     </joint>
   </xacro:macro>

File: reusnake_visualize/urdf/sea_snake.urdf (robot description, URDF)
Before this commit: robot snake, 43 links, 42 joints
Links:
- link joint10__INPUT_INTERFACE: geometry collision cylinder length=-0.033 radius=0.026; visual mesh filename=package://reusnake_visualize/meshes/rotary_input.stl
- link joint10__OUTPUT_BODY: geometry collision cylinder length=-0.033 radius=0.026; visual mesh filename=package://reusnake_visualize/meshes/rotary_output.stl
- link joint11__INPUT_INTERFACE: geometry collision cylinder length=-0.033 radius=0.026; visual mesh filename=package://reusnake_visualize/meshes/rotary_input.stl
- link joint11__OUTPUT_BODY: geometry collision cylinder length=-0.033 radius=0.026; visual mesh filename=package://reusnake_visualize/meshes/rotary_output.stl
- link joint12__INPUT_INTERFACE: geometry collision cylinder length=-0.033 radius=0.026; visual mesh filename=package://reusnake_visualize/meshes/rotary_input.stl
- link joint12__OUTPUT_BODY: geometry collision cylinder length=-0.033 radius=0.026; visual mesh filename=package://reusnake_visualize/meshes/rotary_output.stl
- link joint13__INPUT_INTERFACE: geometry collision cylinder length=-0.033 radius=0.026; visual mesh filename=package://reusnake_visualize/meshes/rotary_input.stl
- link joint13__OUTPUT_BODY: geometry collision cylinder length=-0.033 radius=0.026; visual mesh filename=package://reusnake_visualize/meshes/rotary_output.stl
- link joint14__INPUT_INTERFACE: geometry collision cylinder length=-0.033 radius=0.026; visual mesh filename=package://reusnake_visualize/meshes/rotary_input.stl
- link joint14__OUTPUT_BODY: geometry collision cylinder length=-0.033 radius=0.026; visual mesh filename=package://reusnake_visualize/meshes/rotary_output.stl
- link joint1__INPUT_INTERFACE: geometry collision cylinder length=-0.033 radius=0.026; visual mesh filename=package://reusnake_visualize/meshes/rotary_input.stl
- link joint1__OUTPUT_BODY: geometry collision cylinder length=-0.033 radius=0.026; visual mesh filename=package://reusnake_visualize/meshes/rotary_output.stl
- link joint2__INPUT_INTERFACE: geometry collision cylinder length=-0.033 radius=0.026; visual mesh filename=package://reusnake_visualize/meshes/rotary_input.stl
- link joint2__OUTPUT_BODY: geometry collision cylinder length=-0.033 radius=0.026; visual mesh filename=package://reusnake_visualize/meshes/rotary_output.stl
- link joint3__INPUT_INTERFACE: geometry collision cylinder length=-0.033 radius=0.026; visual mesh filename=package://reusnake_visualize/meshes/rotary_input.stl
- link joint3__OUTPUT_BODY: geometry collision cylinder length=-0.033 radius=0.026; visual mesh filename=package://reusnake_visualize/meshes/rotary_output.stl
- link joint4__INPUT_INTERFACE: geometry collision cylinder length=-0.033 radius=0.026; visual mesh filename=package://reusnake_visualize/meshes/rotary_input.stl
- link joint4__OUTPUT_BODY: geometry collision cylinder length=-0.033 radius=0.026; visual mesh filename=package://reusnake_visualize/meshes/rotary_output.stl
- link joint5__INPUT_INTERFACE: geometry collision cylinder length=-0.033 radius=0.026; visual mesh filename=package://reusnake_visualize/meshes/rotary_input.stl
- link joint5__OUTPUT_BODY: geometry collision cylinder length=-0.033 radius=0.026; visual mesh filename=package://reusnake_visualize/meshes/rotary_output.stl
- link joint6__INPUT_INTERFACE: geometry collision cylinder length=-0.033 radius=0.026; visual mesh filename=package://reusnake_visualize/meshes/rotary_input.stl
- link joint6__OUTPUT_BODY: geometry collision cylinder length=-0.033 radius=0.026; visual mesh filename=package://reusnake_visualize/meshes/rotary_output.stl
- link joint7__INPUT_INTERFACE: geometry collision cylinder length=-0.033 radius=0.026; visual mesh filename=package://reusnake_visualize/meshes/rotary_input.stl
- link joint7__OUTPUT_BODY: geometry collision cylinder length=-0.033 radius=0.026; visual mesh filename=package://reusnake_visualize/meshes/rotary_output.stl
- link joint8__INPUT_INTERFACE: geometry collision cylinder length=-0.033 radius=0.026; visual mesh filename=package://reusnake_visualize/meshes/rotary_input.stl
- link joint8__OUTPUT_BODY: geometry collision cylinder length=-0.033 radius=0.026; visual mesh filename=package://reusnake_visualize/meshes/rotary_output.stl
- link joint9__INPUT_INTERFACE: geometry collision cylinder length=-0.033 radius=0.026; visual mesh filename=package://reusnake_visualize/meshes/rotary_input.stl
- link joint9__OUTPUT_BODY: geometry collision cylinder length=-0.033 radius=0.026; visual mesh filename=package://reusnake_visualize/meshes/rotary_output.stl
Joints:
- joint head__OUTPUT_INTERFACE: origin (none) -> xyz=0 0 0 rpy=0 0 1.57079632679
- joint joint1: origin xyz=0 0 0.0366 rpy=0 0 0 -> xyz=0 0 -0.0366 rpy=0 0 0
- joint joint10: origin xyz=0 0 0.0366 rpy=0 0 0 -> xyz=0 0 -0.0366 rpy=0 0 0
- joint joint10__OUTPUT_INTERFACE: origin xyz=0 0 0.0273 rpy=0 0 -1.57075 -> xyz=0 0 -0.0273 rpy=0 0 -1.57075
- joint joint11: origin xyz=0 0 0.0366 rpy=0 0 0 -> xyz=0 0 -0.0366 rpy=0 0 0
- joint joint11__OUTPUT_INTERFACE: origin xyz=0 0 0.0273 rpy=0 0 -1.57075 -> xyz=0 0 -0.0273 rpy=0 0 -1.57075
- joint joint12: origin xyz=0 0 0.0366 rpy=0 0 0 -> xyz=0 0 -0.0366 rpy=0 0 0
- joint joint12__OUTPUT_INTERFACE: origin xyz=0 0 0.0273 rpy=0 0 -1.57075 -> xyz=0 0 -0.0273 rpy=0 0 -1.57075
- joint joint13: origin xyz=0 0 0.0366 rpy=0 0 0 -> xyz=0 0 -0.0366 rpy=0 0 0
- joint joint13__OUTPUT_INTERFACE: origin xyz=0 0 0.0273 rpy=0 0 -1.57075 -> xyz=0 0 -0.0273 rpy=0 0 -1.57075
- joint joint14: origin xyz=0 0 0.0366 rpy=0 0 0 -> xyz=0 0 -0.0366 rpy=0 0 0
- joint joint1__OUTPUT_INTERFACE: origin xyz=0 0 0.0273 rpy=0 0 -1.57075 -> xyz=0 0 -0.0273 rpy=0 0 -1.57075
- joint joint2: origin xyz=0 0 0.0366 rpy=0 0 0 -> xyz=0 0 -0.0366 rpy=0 0 0
- joint joint2__OUTPUT_INTERFACE: origin xyz=0 0 0.0273 rpy=0 0 -1.57075 -> xyz=0 0 -0.0273 rpy=0 0 -1.57075
- joint joint3: origin xyz=0 0 0.0366 rpy=0 0 0 -> xyz=0 0 -0.0366 rpy=0 0 0
- joint joint3__OUTPUT_INTERFACE: origin xyz=0 0 0.0273 rpy=0 0 -1.57075 -> xyz=0 0 -0.0273 rpy=0 0 -1.57075
- joint joint4: origin xyz=0 0 0.0366 rpy=0 0 0 -> xyz=0 0 -0.0366 rpy=0 0 0
- joint joint4__OUTPUT_INTERFACE: origin xyz=0 0 0.0273 rpy=0 0 -1.57075 -> xyz=0 0 -0.0273 rpy=0 0 -1.57075
- joint joint5: origin xyz=0 0 0.0366 rpy=0 0 0 -> xyz=0 0 -0.0366 rpy=0 0 0
- joint joint5__OUTPUT_INTERFACE: origin xyz=0 0 0.0273 rpy=0 0 -1.57075 -> xyz=0 0 -0.0273 rpy=0 0 -1.57075
- joint joint6: origin xyz=0 0 0.0366 rpy=0 0 0 -> xyz=0 0 -0.0366 rpy=0 0 0
- joint joint6__OUTPUT_INTERFACE: origin xyz=0 0 0.0273 rpy=0 0 -1.57075 -> xyz=0 0 -0.0273 rpy=0 0 -1.57075
- joint joint7: origin xyz=0 0 0.0366 rpy=0 0 0 -> xyz=0 0 -0.0366 rpy=0 0 0
- joint joint7__OUTPUT_INTERFACE: origin xyz=0 0 0.0273 rpy=0 0 -1.57075 -> xyz=0 0 -0.0273 rpy=0 0 -1.57075
- joint joint8: origin xyz=0 0 0.0366 rpy=0 0 0 -> xyz=0 0 -0.0366 rpy=0 0 0
- joint joint8__OUTPUT_INTERFACE: origin xyz=0 0 0.0273 rpy=0 0 -1.57075 -> xyz=0 0 -0.0273 rpy=0 0 -1.57075
- joint joint9: origin xyz=0 0 0.0366 rpy=0 0 0 -> xyz=0 0 -0.0366 rpy=0 0 0
- joint joint9__OUTPUT_INTERFACE: origin xyz=0 0 0.0273 rpy=0 0 -1.57075 -> xyz=0 0 -0.0273 rpy=0 0 -1.57075

File: reusnake_visualize/urdf/sea_snake.urdf.xacro (robot description, xacro)
@@ -27,5 +27,5 @@
     <parent link="link0"/>
     <child link="${S_00}__INPUT_INTERFACE"/>
-    <!-- <origin xyz="${width/2} ${leg_y_offset} ${height/2}" rpy="-${PI/2} 0 -${PI/2}"/> -->
+    <origin xyz="0 0 0" rpy="0 0 ${PI/2}"/>
   </joint>
   <xacro:rotary_module joint="${S_00}" child="${S_01}"/>
