Commit message: urdf change

File: reusnake_visualize/urdf/sea_snake.urdf (robot description, URDF)
Before this commit: robot snake, 43 links, 42 joints
Links:
- removed link joint13__INPUT_INTERFACE
- removed link joint13__INPUT_INTERFACE__COLLAR
- removed link joint13__OUTPUT_BODY
- removed link joint14__INPUT_INTERFACE
- removed link joint14__INPUT_INTERFACE__COLLAR
- removed link joint14__OUTPUT_BODY
Joints:
- removed joint joint12__OUTPUT_INTERFACE
- removed joint joint13
- removed joint joint13__INPUT_INTERFACE__COLLAR_JOINT
- removed joint joint13__OUTPUT_INTERFACE
- removed joint joint14
- removed joint joint14__INPUT_INTERFACE__COLLAR_JOINT
- joint head__OUTPUT_INTERFACE: origin xyz=0 0 0 rpy=0 0 1.57079632679 -> xyz=0 0 0 rpy=0 0 -1.57079632679

File: reusnake_visualize/urdf/sea_snake.urdf.xacro (robot description, xacro)
@@ -27,5 +27,5 @@
     <parent link="link0"/>
     <child link="${S_00}__INPUT_INTERFACE"/>
-    <origin xyz="0 0 0" rpy="0 0 ${PI/2}"/>
+    <origin xyz="0 0 0" rpy="0 0 -${PI/2}"/>
   </joint>
   <xacro:rotary_module joint="${S_00}" child="${S_01}"/>
@@ -40,12 +40,14 @@
   <xacro:rotary_module joint="${S_09}" child="${S_10}"/>
   <xacro:rotary_module joint="${S_10}" child="${S_11}"/>
+  <!--
   <xacro:rotary_module joint="${S_11}" child="${S_12}"/>
   <xacro:rotary_module joint="${S_12}" child="${S_13}"/>
+  -->
   <!-- first half of joint + collar -->
-  <xacro:rotary_module_in name="${S_13}__INPUT_INTERFACE"/>
-  <xacro:collar parent="${S_13}__INPUT_INTERFACE"/>
+  <xacro:rotary_module_in name="${S_11}__INPUT_INTERFACE"/>
+  <xacro:collar parent="${S_11}__INPUT_INTERFACE"/>
   <!-- actual rotary joint component: -->
-  <xacro:rotary_module_joint parent="${S_13}__INPUT_INTERFACE" name="${S_13}" child="${S_13}__OUTPUT_BODY"/>
+  <xacro:rotary_module_joint parent="${S_11}__INPUT_INTERFACE" name="${S_11}" child="${S_11}__OUTPUT_BODY"/>
   <!-- second half of joint -->
-  <xacro:rotary_module_out name="${S_13}__OUTPUT_BODY"/>
+  <xacro:rotary_module_out name="${S_11}__OUTPUT_BODY"/>
 </robot>

Commit message: Updated visualization to plot gazebo ground truth

File: reusnake_visualize/urdf/sea_snake.urdf (robot description, URDF)
Before this commit: robot snake, 37 links, 36 joints
Links:
- added link joint13__INPUT_INTERFACE, mass 0.103; collision cylinder length=-0.033 radius=0.026; visual mesh filename=package://reusnake_visualize/meshes/rotary_input.stl
- added link joint13__INPUT_INTERFACE__COLLAR; visual cylinder length=0.01 radius=0.026
- added link joint13__OUTPUT_BODY, mass 0.103; collision cylinder length=-0.033 radius=0.026; visual mesh filename=package://reusnake_visualize/meshes/rotary_output.stl
- added link joint14__INPUT_INTERFACE, mass 0.103; collision cylinder length=-0.033 radius=0.026; visual mesh filename=package://reusnake_visualize/meshes/rotary_input.stl
- added link joint14__INPUT_INTERFACE__COLLAR; visual cylinder length=0.01 radius=0.026
- added link joint14__OUTPUT_BODY, mass 0.103; collision cylinder length=-0.033 radius=0.026; visual mesh filename=package://reusnake_visualize/meshes/rotary_output.stl
- added link joint15__INPUT_INTERFACE, mass 0.103; collision cylinder length=-0.033 radius=0.026; visual mesh filename=package://reusnake_visualize/meshes/rotary_input.stl
- added link joint15__INPUT_INTERFACE__COLLAR; visual cylinder length=0.01 radius=0.026
- added link joint15__OUTPUT_BODY, mass 0.103; collision cylinder length=-0.033 radius=0.026; visual mesh filename=package://reusnake_visualize/meshes/rotary_output.stl
- added link joint16__INPUT_INTERFACE, mass 0.103; collision cylinder length=-0.033 radius=0.026; visual mesh filename=package://reusnake_visualize/meshes/rotary_input.stl
- added link joint16__INPUT_INTERFACE__COLLAR; visual cylinder length=0.01 radius=0.026
- added link joint16__OUTPUT_BODY, mass 0.103; collision cylinder length=-0.033 radius=0.026; visual mesh filename=package://reusnake_visualize/meshes/rotary_output.stl
Joints:
- added joint joint12__OUTPUT_INTERFACE: type fixed, parent joint12__OUTPUT_BODY, child joint13__INPUT_INTERFACE, origin xyz=0 0 -0.0273 rpy=0 0 -1.57075
- added joint joint13: type revolute, parent joint13__INPUT_INTERFACE, child joint13__OUTPUT_BODY, origin xyz=0 0 -0.0366 rpy=0 0 0, axis 0 1 0, limit lower=-1.57 upper=1.57 effort=7.0 velocity=2.208932
- added joint joint13__INPUT_INTERFACE__COLLAR_JOINT: type fixed, parent joint13__INPUT_INTERFACE, child joint13__INPUT_INTERFACE__COLLAR
- added joint joint13__OUTPUT_INTERFACE: type fixed, parent joint13__OUTPUT_BODY, child joint14__INPUT_INTERFACE, origin xyz=0 0 -0.0273 rpy=0 0 -1.57075
- added joint joint14: type revolute, parent joint14__INPUT_INTERFACE, child joint14__OUTPUT_BODY, origin xyz=0 0 -0.0366 rpy=0 0 0, axis 0 1 0, limit lower=-1.57 upper=1.57 effort=7.0 velocity=2.208932
- added joint joint14__INPUT_INTERFACE__COLLAR_JOINT: type fixed, parent joint14__INPUT_INTERFACE, child joint14__INPUT_INTERFACE__COLLAR
- added joint joint14__OUTPUT_INTERFACE: type fixed, parent joint14__OUTPUT_BODY, child joint15__INPUT_INTERFACE, origin xyz=0 0 -0.0273 rpy=0 0 -1.57075
- added joint joint15: type revolute, parent joint15__INPUT_INTERFACE, child joint15__OUTPUT_BODY, origin xyz=0 0 -0.0366 rpy=0 0 0, axis 0 1 0, limit lower=-1.57 upper=1.57 effort=7.0 velocity=2.208932
- added joint joint15__INPUT_INTERFACE__COLLAR_JOINT: type fixed, parent joint15__INPUT_INTERFACE, child joint15__INPUT_INTERFACE__COLLAR
- added joint joint15__OUTPUT_INTERFACE: type fixed, parent joint15__OUTPUT_BODY, child joint16__INPUT_INTERFACE, origin xyz=0 0 -0.0273 rpy=0 0 -1.57075
- added joint joint16: type revolute, parent joint16__INPUT_INTERFACE, child joint16__OUTPUT_BODY, origin xyz=0 0 -0.0366 rpy=0 0 0, axis 0 1 0, limit lower=-1.57 upper=1.57 effort=7.0 velocity=2.208932
- added joint joint16__INPUT_INTERFACE__COLLAR_JOINT: type fixed, parent joint16__INPUT_INTERFACE, child joint16__INPUT_INTERFACE__COLLAR
